File: testfixture/testfixture.sch (KiCad schematic (older format))
At the start: 3 parts, among them J101 Conn_Coaxial, J102 Conn_Coaxial, J103 632712000011

Commit message: Rev.B
Parts:
- J103: symbol wue:632712000011 -> testfixture-rescue:632712000011-wue
Changed lines of the file:
@@
 $EndComp
 $Comp
-L wue:632712000011 J103
+L testfixture-rescue:632712000011-wue J103
 U 1 1 5FFE2B8F
 P 6150 2500
