File: testfixture/testfixture.sch (KiCad schematic (older format))
At the start: 3 parts, among them J101 Conn_Coaxial, J102 Conn_Coaxial, J103 632712000011

Commit message: Rev.B with Resistors and 45 Ohm matching
Parts:
- added R101, R102, R103, R104: R, Resistor_SMD:R_0402_1005Metric, symbol Device:R
- J103: symbol wue:632712000011 -> testfixture-rescue:632712000011-wue
Connections:
- net GND: now also R101.2, R102.2
- net at J101.1 (In): now also R103.1; no longer J103.A6 (DP1)
- net at J103.A7 (DN1): now also R102.1, R104.2; no longer J102.1 (In)
- new net: J103.A6 (DP1), R101.1, R103.2
- new net: J102.1 (In), R104.1
Changed lines of the file:
@@
 $EndComp
 $Comp
-L wue:632712000011 J103
+L testfixture-rescue:632712000011-wue J103
 U 1 1 5FFE2B8F
 P 6150 2500
@@
 	1    0    0    -1
 $EndComp
-Wire Wire Line
-	5450 2400 3750 2400
-Wire Wire Line
-	3750 2400 3750 2350
-Wire Wire Line
-	5450 2500 3750 2500
-Wire Wire Line
-	3750 2500 3750 3050
 $Comp
-L power:GND #PWR?
+L power:GND #PWR0103
 U 1 1 5FFF7EB2
 P 5450 3100
-F 0 "#PWR?" H 5450 2850 50  0001 C CNN
+F 0 "#PWR0103" H 5450 2850 50  0001 C CNN
 F 1 "GND" H 5455 2927 50  0000 C CNN
 F 2 "" H 5450 3100 50  0001 C CNN
@@
 $EndComp
 $Comp
-L power:GND #PWR?
+L power:GND #PWR0104
 U 1 1 5FFF9496
 P 6850 3100
-F 0 "#PWR?" H 6850 2850 50  0001 C CNN
+F 0 "#PWR0104" H 6850 2850 50  0001 C CNN
 F 1 "GND" H 6855 2927 50  0000 C CNN
 F 2 "" H 6850 3100 50  0001 C CNN
@@
 	1    0    0    -1
 $EndComp
+$Comp
+L Device:R R101
+U 1 1 62CCD558
+P 4700 2500
+F 0 "R101" H 4770 2546 50  0000 L CNN
+F 1 "R" H 4770 2455 50  0000 L CNN
+F 2 "Resistor_SMD:R_0402_1005Metric" V 4630 2500 50  0001 C CNN
+F 3 "~" H 4700 2500 50  0001 C CNN
+	1    4700 2500
+	1    0    0    -1
+$EndComp
+$Comp
+L Device:R R102
+U 1 1 62CCDF6E
+P 4700 3200
+F 0 "R102" H 4770 3246 50  0000 L CNN
+F 1 "R" H 4770 3155 50  0000 L CNN
+F 2 "Resistor_SMD:R_0402_1005Metric" V 4630 3200 50  0001 C CNN
+F 3 "~" H 4700 3200 50  0001 C CNN
+	1    4700 3200
+	1    0    0    -1
+$EndComp
+$Comp
+L Device:R R103
+U 1 1 62CCE2E6
+P 4450 2350
+F 0 "R103" V 4657 2350 50  0000 C CNN
+F 1 "R" V 4566 2350 50  0000 C CNN
+F 2 "Resistor_SMD:R_0402_1005Metric" V 4380 2350 50  0001 C CNN
+F 3 "~" H 4450 2350 50  0001 C CNN
+	1    4450 2350
+	0    -1   -1   0
+$EndComp
+$Comp
+L Device:R R104
+U 1 1 62CCE840
+P 4450 3050
+F 0 "R104" V 4657 3050 50  0000 C CNN
+F 1 "R" V 4566 3050 50  0000 C CNN
+F 2 "Resistor_SMD:R_0402_1005Metric" V 4380 3050 50  0001 C CNN
+F 3 "~" H 4450 3050 50  0001 C CNN
+	1    4450 3050
+	0    -1   -1   0
+$EndComp
+$Comp
+L power:GND #PWR0105
+U 1 1 62CCECF0
+P 4700 3350
+F 0 "#PWR0105" H 4700 3100 50  0001 C CNN
+F 1 "GND" H 4705 3177 50  0000 C CNN
+F 2 "" H 4700 3350 50  0001 C CNN
+F 3 "" H 4700 3350 50  0001 C CNN
+	1    4700 3350
+	1    0    0    -1
+$EndComp
+$Comp
+L power:GND #PWR0106
+U 1 1 62CCF06A
+P 4700 2650
+F 0 "#PWR0106" H 4700 2400 50  0001 C CNN
+F 1 "GND" H 4705 2477 50  0000 C CNN
+F 2 "" H 4700 2650 50  0001 C CNN
+F 3 "" H 4700 2650 50  0001 C CNN
+	1    4700 2650
+	1    0    0    -1
+$EndComp
+Wire Wire Line
+	3750 2350 4100 2350
+Wire Wire Line
+	4100 2350 4300 2350
+Connection ~ 4100 2350
+Wire Wire Line
+	4600 2350 4700 2350
+Wire Wire Line
+	5250 2350 5250 2400
+Wire Wire Line
+	5250 2400 5450 2400
+Wire Wire Line
+	5450 2500 5200 2500
+Wire Wire Line
+	5200 2500 5200 3050
+Wire Wire Line
+	5200 3050 4700 3050
+Wire Wire Line
+	4300 3050 4100 3050
+Wire Wire Line
+	3750 3050 4100 3050
+Connection ~ 4100 3050
+Connection ~ 4700 2350
+Wire Wire Line
+	4700 2350 5250 2350
+Connection ~ 4700 3050
+Wire Wire Line
+	4700 3050 4600 3050
 $EndSCHEMATC
